File: hardware/BREAD_Slice.kicad_pcb (KiCad board)
At the start: 2 copper layers, 72.6 x 100 mm, 16 parts, among them J1 Conn_01x10_Female, J2 I2C_01x04

Commit message: finished first pass of schematic and board
Parts:
- added C14: 10u, Capacitor_SMD:C_0805_2012Metric_Pad1.18x1.45mm_HandSolder, B.Cu at (138.3, 79.8)
- added C15: 10n, Capacitor_SMD:C_0805_2012Metric_Pad1.18x1.45mm_HandSolder, B.Cu at (137.2, 82.8)
- added C16: 10n, Capacitor_SMD:C_0805_2012Metric_Pad1.18x1.45mm_HandSolder, B.Cu at (151.7, 80.6)
- added C17: 10u, Capacitor_SMD:C_0805_2012Metric_Pad1.18x1.45mm_HandSolder, B.Cu at (149.2, 76.4)
- added C5: 0.1u, Capacitor_SMD:C_0603_1608Metric_Pad1.08x0.95mm_HandSolder, F.Cu at (180.2, 82.2)
- added C6: 10n, Capacitor_SMD:C_0603_1608Metric_Pad1.08x0.95mm_HandSolder, F.Cu at (175.8, 87.1)
- added C7: 10n, Capacitor_SMD:C_0603_1608Metric_Pad1.08x0.95mm_HandSolder, F.Cu at (175.7, 76.8)
- added C8: 10n, Capacitor_SMD:C_0603_1608Metric_Pad1.08x0.95mm_HandSolder, F.Cu at (179.1, 87.1)
- added C9: 10n, Capacitor_SMD:C_0603_1608Metric_Pad1.08x0.95mm_HandSolder, F.Cu at (179.1, 76.8)
- added J3: Screw_Terminal_01x05, TerminalBlock_4Ucon:TerminalBlock_4Ucon_1x05_P3.50mm_Horizontal, F.Cu at (188.2, 67.4)
- added J4: Screw_Terminal_01x05, TerminalBlock_4Ucon:TerminalBlock_4Ucon_1x05_P3.50mm_Horizontal, F.Cu at (188.2, 105.8)
- added J5: Screw_Terminal_01x05, TerminalBlock_4Ucon:TerminalBlock_4Ucon_1x05_P3.50mm_Horizontal, F.Cu at (188.2, 86.6)
- added NT1: NetTie_2, NetTie:NetTie-2_SMD_Pad2.0mm, B.Cu at (128.7, 115.2)
- added NT2: NetTie_2, NetTie:NetTie-2_SMD_Pad2.0mm, B.Cu at (142.7, 87.5)
- added R1: 1k, Resistor_SMD:R_0603_1608Metric_Pad0.98x0.95mm_HandSolder, F.Cu at (174.8, 89.5)
- added R10: 99, Resistor_SMD:R_0805_2012Metric_Pad1.20x1.40mm_HandSolder, B.Cu at (149.1, 84.8)
- added R2: 1k, Resistor_SMD:R_0603_1608Metric_Pad0.98x0.95mm_HandSolder, F.Cu at (174.8, 74.4)
- added R3: 1k, Resistor_SMD:R_0603_1608Metric_Pad0.98x0.95mm_HandSolder, F.Cu at (178.2, 89.5)
- added R4: 1k, Resistor_SMD:R_0603_1608Metric_Pad0.98x0.95mm_HandSolder, F.Cu at (178.1, 74.4)
- added R5: 1k, Resistor_SMD:R_0603_1608Metric_Pad0.98x0.95mm_HandSolder, F.Cu at (176.7, 89.5)
- added R6: 1k, Resistor_SMD:R_0603_1608Metric_Pad0.98x0.95mm_HandSolder, F.Cu at (176.6, 74.4)
- added R7: 1k, Resistor_SMD:R_0603_1608Metric_Pad0.98x0.95mm_HandSolder, F.Cu at (180.0, 89.5)
- added R8: 1k, Resistor_SMD:R_0603_1608Metric_Pad0.98x0.95mm_HandSolder, F.Cu at (180.0, 74.4)
- added R9: 99, Resistor_SMD:R_0805_2012Metric_Pad1.20x1.40mm_HandSolder, B.Cu at (149.1, 80.6)
- added U2: ADS1234IPW, Package_SO:TSSOP-28_4.4x9.7mm_P0.65mm, F.Cu at (174.2, 82.0)
- added U3: TPS7A4901DGNR, kml-custom:DGN8_1P89X1P57, B.Cu at (143.8, 81.7)
- HS1: footprint SparkFun-Fuse:Thermal Pad -> kml-custom:Thermal Pad
- J2: value I2C_01x04 -> Screw_Terminal_01x05; footprint Connector_JST:JST_SH_SM04B-SRSS-TB_1x04-1MP_P1.00mm_Horizontal -> TerminalBlock_4Ucon:TerminalBlock_4Ucon_1x05_P3.50mm_Horizontal; moved to F.Cu
- U1: value ~ -> AP63205
- moved J2 39.7 mm to (188.2, 125.0), turned to 90 degrees
- moved A1 2.56 mm to (142.6, 97.4)
- moved Logo1 1.57 mm to (128.2, 71.9)
- moved HS1 0.46 mm to (131.8, 121.5)
- moved D1 0.45 mm to (173.1, 135.7)
- moved C1 0.25 mm to (128.8, 119.5)
- moved C4 0.05 mm to (133.8, 116.4)
Connections:
- net /E_STOP renamed /ESTOP
- A1 pad 10: unconnected-(A1-D7-Pad10) -> /GAIN_SEL_0
- A1 pad 11: unconnected-(A1-D8-Pad11) -> /CH_SEL_0
- A1 pad 12: unconnected-(A1-D9-Pad12) -> /CH_SEL_1
- A1 pad 13: unconnected-(A1-D10-Pad13) -> /SPEED
- A1 pad 14: unconnected-(A1-D11-Pad14) -> /PWDN
- A1 pad 15: unconnected-(A1-D12-Pad15) -> /MISO
- A1 pad 16: unconnected-(A1-D13-Pad16) -> /SCK
- A1 pad 9: unconnected-(A1-D6-Pad9) -> /GAIN_SEL_1
- J1 pad 1: GND -> GNDPWR
- J1 pad 10: GND -> GNDPWR
- J1 pad 5: GND -> GNDPWR
- J2 pad 1: GND -> GNDA
- J2 pad 2: +5V -> /SIG1+
- J2 pad 3: /I2C_DAT -> /SIG1-
- J2 pad 4: /I2C_CLK -> GNDA
Routing:
- net +5VA: track 0.00 -> 103.0 mm, vias 0 -> 1
- net /PWDN: track 0.00 -> 68.1 mm, vias 0 -> 1
- net /MISO: track 0.00 -> 67.4 mm, vias 0 -> 1
- net /SPEED: track 0.00 -> 67.0 mm, vias 0 -> 1
- net /CH_SEL_1: track 0.00 -> 63.9 mm, vias 0 -> 1
- net /SCK: track 0.00 -> 63.8 mm, vias 0 -> 1
- net /CH_SEL_0: track 0.00 -> 63.3 mm, vias 0 -> 1
- net /GAIN_SEL_0: track 0.00 -> 61.7 mm, vias 0 -> 1
- net /GAIN_SEL_1: track 0.00 -> 60.1 mm, vias 0 -> 1
- net GNDPWR: track 0.00 -> 43.7 mm
- net /LED: track 51.5 -> 92.9 mm
- net /SIG1+: track 0.00 -> 36.6 mm
- net +12V: track 46.8 -> 81.4 mm, vias 0 -> 1
- net /SIG1-: track 0.00 -> 32.4 mm
- net /I2C_CLK: track 78.5 -> 46.3 mm, vias 2 -> 0
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- added copper zone on B.Cu, net GNDA
- added copper zone on B.Cu, net GNDPWR
Other:
- board size 72.6 x 100 mm -> 70 x 100 mm
- board text added: "BREAD Slice Load Cell Amps SLC_LOAD R3 04-2025"
- board text removed: "5V I2C Connector"
- board text removed: "BREAD Slice Template SLC_TEMP <version> <year>"
