File: hardware/BREAD_Slice.kicad_sch (KiCad schematic)
At the start: 15 parts, among them J1 Conn_01x10_Female, J2 I2C_01x04

Commit message: finished first pass of schematic and board
Parts:
- removed J2: I2C_01x04, Connector_JST:JST_SH_SM04B-SRSS-TB_1x04-1MP_P1.00mm_Horizontal, symbol SparkFun-Connector:I2C_01x04
- added J2, J3, J4, J5: Screw_Terminal_01x05, TerminalBlock_4Ucon:TerminalBlock_4Ucon_1x05_P3.50mm_Horizontal, symbol Connector:Screw_Terminal_01x05
- added NT1: NetTie_2, NetTie:NetTie-2_SMD_Pad2.0mm, symbol Device:NetTie_2
- added RSG1, RSG2, RSG3, RSG4: 350, symbol kml-custom:Full_Bridge_Strain_Gauge
- D1: PROD_ID (none) -> DIO-12503
- HS1: footprint SparkFun-Fuse:Thermal Pad -> kml-custom:Thermal Pad
- U1: value ~ -> AP63205
Connections:
- net GND: now also NT1.1; no longer J1.1 (Pin_1), J1.10 (Pin_10), J1.5 (Pin_5)
- net GAIN_SEL_0: now reaches A1.10 (D7)
- net CH_SEL_0: now reaches A1.11 (D8)
- net CH_SEL_1: now reaches A1.12 (D9)
- net SPEED: now reaches A1.13 (D10)
- net PWDN: now reaches A1.14 (D11)
- net MISO: now reaches A1.15 (D12)
- net SCK: now reaches A1.16 (D13)
- net GAIN_SEL_1: now reaches A1.9 (D6)
- net E_STOP renamed ESTOP
- new net +5VA: J2.5 (Pin_5), J3.1 (Pin_1), J4.5 (Pin_5), J5.1 (Pin_1), RSG1.1 (EXC+), RSG2.1 (EXC+), RSG3.1 (EXC+), RSG4.1 (EXC+)
- new net GNDA: J2.1 (Pin_1), J2.4 (Pin_4), J3.2 (Pin_2), J3.5 (Pin_5), J4.1 (Pin_1), J4.4 (Pin_4), J5.2 (Pin_2), J5.5 (Pin_5), RSG1.2 (EXC-), RSG2.2 (EXC-), RSG3.2 (EXC-), RSG4.2 (EXC-)
- new net GNDPWR: J1.1 (Pin_1), J1.10 (Pin_10), J1.5 (Pin_5), NT1.2
- new net SIG1+: J2.2 (Pin_2), RSG1.3 (SIG+)
- new net SIG1-: J2.3 (Pin_3), RSG1.4 (SIG-)
- new net SIG2+: J3.4 (Pin_4), RSG2.3 (SIG+)
- new net SIG2-: J3.3 (Pin_3), RSG2.4 (SIG-)
- new net SIG3+: J4.2 (Pin_2), RSG3.3 (SIG+)
- new net SIG3-: J4.3 (Pin_3), RSG3.4 (SIG-)
- new net SIG4+: J5.4 (Pin_4), RSG4.3 (SIG+)
- new net SIG4-: J5.3 (Pin_3), RSG4.4 (SIG-)
- no-connect marks 22 -> 14
Other:
- added sheet Strain Gauge ADC 4-Ch (ads1234.kicad_sch)
- added sheet TPS7A4901-5VA (tps7a4901.kicad_sch)
- note added: "5V Switching Supply"
- note added: "A+"
- note added: "A-"
- note added: "ADS1234 4-Channel ADC for Bridge Sensors"
- note added: "Analog 5V"
- note added: "Arduino Nano"
- note added: "Backplane Conn."
- note added: "Black"
- note added: "Clean 5V for analog frontend"
- note added: "Color Scheme Legend: ---------------------------------------------------------- color - value - reference ---------------------------------------------------------- • Red - red3 - Analog 5V Supply (e.g., for amps, ADC, references) • Brown - orange1 - Analog Ground (sensor/amp/ADC ground) • Orange - orange3 - Digital 5V Supply (MCU, digital circuits) • Black - black - Digital Ground (MCU ground) •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"
- note added: "Common Load Cell Colors:"
- note added: "E+"
- note added: "E-"
- note added: "Green or Blue"
- note added: "Load Cells"
- note added: "Mounting Holes"
- note added: "Pinout Details Arduino Nano: -------------------------------------------------------------------------------------------------------------------- Pin | Function | Limitations/Notes -------------------------------------------------------------------------------------------------------------------- VIN | External Supply Input | External power source 7-12V GND | Ground | First GND pin available for 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"
- note added: "RGB LED"
- note added: "Red"
- note added: "Shield"
- note added: "Terminal Connectors"
- note added: "White"
- note added: "Yellow"
- moved on the sheet: A1, C1, C2, C3, C4, H1, H2, H3, H4, L1, U1

Commit message: minor tweaks
Other:
- note added: "Red Black White Green/Blue Yellow"
- note removed: "Black"
- note removed: "Green or Blue"
- note removed: "Red"
- note removed: "White"
- note removed: "Yellow"
Changed lines of the file:
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@@
-		)
-	)
-	(text "Red"
-		(exclude_from_sim no)
-		(at 123.19 52.07 0)
-		(effects
-			(font
-				(size 1.778 1.5113)
-			)
-			(justify left bottom)
 		)
 	)
@@
 	(text "Common Load\nCell Colors:"
 		(exclude_from_sim no)
-		(at 115.824 45.974 0)
-		(effects
-			(font
-				(size 1.778 1.5113)
+		(at 119.38 46.99 0)
+		(effects
+			(font
+				(size 1.778 1.5113)
+				(thickness 0.3023)
+				(bold yes)
 			)
 			(justify left bottom)
@@
 		)
 	)
-	(text "White"
-		(exclude_from_sim no)
-		(at 123.19 57.15 0)
-		(effects
-			(font
-				(size 1.778 1.5113)
-			)
-			(justify left bottom)
-		)
-	)
 	(text "Color Scheme Legend:\n----------------------------------------------------------\ncolor		-	value		-	reference\n----------------------------------------------------------\n• Red		-	red3		-	Analog 5V Supply (e.g., for amps, ADC, references)\n• Brown		-	orange1		-	Analog Ground (sensor/amp/ADC ground)\n• Orange	-	orange3		-	Digital 5V Supply (MCU, digital circuits)\n• Black		-	black		-	Digital Ground (MCU ground)\n• Pink		-	magenta3	-	12V Source Supply (from 12V rail on backplane)\n• Blue		-	blue3		-	Clock Signals (oscillator, ADC CLKIN, SPI SCLK)\n• Green		-	green3		-	Analog Signals (amp outputs to ADC + inputs)\n• Yellow	-	yellow3		-	SPI Control (CS, SYNC/RESET, etc.)\n• Purple	-	#A020F0		-	Special/Reference/Control Signals\n• Grey		-	gray2		-	Miscellaneous/Unassigned\n• Teal		-	cyan2		-	Template/Backplane Connections\n----------------------------------------------------------"
 		(exclude_from_sim no)
@@
 		)
 	)
-	(text "Green or Blue"
-		(exclude_from_sim no)
-		(at 113.03 59.69 0)
-		(effects
-			(font
-				(size 1.778 1.5113)
-			)
-			(justify left bottom)
-		)
-	)
 	(text "E-"
 		(exclude_from_sim no)
@@
 		(exclude_from_sim no)
 		(at 135.89 62.23 0)
-		(effects
-			(font
-				(size 1.778 1.5113)
-			)
-			(justify left bottom)
-		)
-	)
-	(text "Yellow"
-		(exclude_from_sim no)
-		(at 123.19 62.23 0)
 		(effects
 			(font
@@
 		)
 	)
-	(text "Black"
-		(exclude_from_sim no)
-		(at 123.19 54.61 0)
-		(effects
-			(font
-				(size 1.778 1.5113)
-			)
-			(justify left bottom)
-		)
-	)
 	(text "Core Slice Components"
 		(exclude_from_sim no)
@@
 		(effects
 			(font
+				(size 1.778 1.5113)
+			)
+			(justify left bottom)
+		)
+	)
+	(text "Red\nBlack\nWhite\nGreen/Blue\nYellow"
+		(exclude_from_sim no)
+		(at 119.634 62.738 0)
+		(effects
+			(font
