File: hardware/ads1234.kicad_sch (KiCad schematic)
At the start: 14 parts, among them U2 ADS1234IPW

Commit message: chore: minor updates
Parts:
- added C5: 0.1u, Capacitor_SMD:C_0603_1608Metric_Pad1.08x0.95mm_HandSolder, symbol Device:C
- renumbered C9 to C10, C5 to C6, C6 to C7, C7 to C8, C8 to C9, R5 to R2, R2 to R3, R6 to R4, R3 to R5, R7 to R6, R4 to R7
Connections:
- net +5VA: now also C5.2
- net GNDA: now also C5.1
Changed lines of the file:
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@@
+	)
+	(junction
+		(at 63.5 31.75)
+		(diameter 0)
+		(color 194 0 0 1)
 	)
 	(junction
@@
 	(wire
 		(pts
+			(xy 63.5 44.45) (xy 63.5 39.37)
+		)
+		(stroke
+			(width 0.2032)
+			(type default)
+			(color 128 77 0 1)
+		)
+	)
+	(wire
+		(pts
 			(xy 135.89 170.18) (xy 128.27 170.18)
 		)
@@
 	(wire
 		(pts
-			(xy 49.53 31.75) (xy 77.47 31.75)
+			(xy 49.53 31.75) (xy 63.5 31.75)
 		)
 		(stroke
@@
 	(wire
 		(pts
+			(xy 63.5 31.75) (xy 77.47 31.75)
+		)
+		(stroke
+			(width 0.2032)
+			(type default)
+			(color 194 0 0 1)
+		)
+	)
+	(wire
+		(pts
 			(xy 156.21 52.07) (xy 119.38 52.07)
 		)
@@
 	(label "IN2-"
 		(at 63.5 67.31 180)
+		(effects
+			(font
+				(size 1.27 1.27)
+			)
+			(justify right bottom)
+		)
+	)
+	(label "GNDA"
+		(at 63.5 44.45 180)
 		(effects
 			(font
@@
 		(on_board yes)
 		(dnp no)
-		(property "Reference" "R3"
+		(property "Reference" "R5"
 			(at 122.428 138.43 90)
 			(effects
@@
 			(project "BREAD_Slice"
 				(path "/66043bca-a260-4915-9fce-8a51d324c687/750db89f-8b40-4cde-930a-58e7ceb323d5"
-					(reference "R3")
+					(reference "R5")
 					(unit 1)
 				)
@@
 		(on_board yes)
 		(dnp no)
-		(property "Reference" "C6"
+		(property "Reference" "C7"
 			(at 91.44 147.32 0)
 			(effects
@@
 			(project "BREAD_Slice"
 				(path "/66043bca-a260-4915-9fce-8a51d324c687/750db89f-8b40-4cde-930a-58e7ceb323d5"
-					(reference "C6")
+					(reference "C7")
 					(unit 1)
 				)
@@
 		(on_board yes)
 		(dnp no)
-		(property "Reference" "R6"
+		(property "Reference" "R4"
 			(at 80.518 185.42 90)
 			(effects
@@
 			(project "BREAD_Slice"
 				(path "/66043bca-a260-4915-9fce-8a51d324c687/750db89f-8b40-4cde-930a-58e7ceb323d5"
-					(reference "R6")
+					(reference "R4")
 					(unit 1)
 				)
@@
 		(on_board yes)
 		(dnp no)
-		(property "Reference" "R2"
+		(property "Reference" "R3"
 			(at 80.518 165.1 90)
 			(effects
@@
 			(project "BREAD_Slice"
 				(path "/66043bca-a260-4915-9fce-8a51d324c687/750db89f-8b40-4cde-930a-58e7ceb323d5"
-					(reference "R2")
+					(reference "R3")
 					(unit 1)
 				)
@@
 		(on_board yes)
 		(dnp no)
-		(property "Reference" "C9"
+		(property "Reference" "C10"
 			(at 133.35 173.99 0)
 			(effects
@@
 			(project "BREAD_Slice"
 				(path "/66043bca-a260-4915-9fce-8a51d324c687/750db89f-8b40-4cde-930a-58e7ceb323d5"
-					(reference "C9")
+					(reference "C10")
 					(unit 1)
 				)
@@
 		(on_board yes)
 		(dnp no)
-		(property "Reference" "C7"
+		(property "Reference" "C8"
 			(at 91.44 173.99 0)
 			(effects
@@
 			(project "BREAD_Slice"
 				(path "/66043bca-a260-4915-9fce-8a51d324c687/750db89f-8b40-4cde-930a-58e7ceb323d5"
-					(reference "C7")
+					(reference "C8")
 					(unit 1)
 				)
@@
 		(on_board yes)
 		(dnp no)
-		(property "Reference" "C5"
+		(property "Reference" "C6"
 			(at 74.93 42.926 90)
 			(effects
@@
 			(project ""
 				(path "/66043bca-a260-4915-9fce-8a51d324c687/750db89f-8b40-4cde-930a-58e7ceb323d5"
-					(reference "C5")
+					(reference "C6")
 					(unit 1)
 				)
@@
 		(on_board yes)
 		(dnp no)
-		(property "Reference" "C8"
+		(property "Reference" "C9"
 			(at 133.35 147.32 0)
 			(effects
@@
 			(project "BREAD_Slice"
 				(path "/66043bca-a260-4915-9fce-8a51d324c687/750db89f-8b40-4cde-930a-58e7ceb323d5"
-					(reference "C8")
+					(reference "C9")
 					(unit 1)
 				)
@@
 		(on_board yes)
 		(dnp no)
-		(property "Reference" "R5"
+		(property "Reference" "R2"
 			(at 80.518 158.75 90)
 			(effects
@@
 			(project "BREAD_Slice"
 				(path "/66043bca-a260-4915-9fce-8a51d324c687/750db89f-8b40-4cde-930a-58e7ceb323d5"
-					(reference "R5")
+					(reference "R2")
 					(unit 1)
 				)
@@
 	)
 	(symbol
+		(lib_id "Device:C")
+		(at 63.5 35.56 180)
+		(unit 1)
+		(exclude_from_sim no)
+		(in_bom yes)
+		(on_board yes)
+		(dnp no)
+		(property "Reference" "C5"
+			(at 58.42 34.544 0)
+			(effects
+				(font
+					(size 1.27 1.27)
+				)
+			)
+		)
+		(property "Value" "0.1u"
+			(at 58.674 36.576 0)
+			(effects
+				(font
+					(size 1.27 1.27)
+				)
+			)
+		)
+		(property "Footprint" "Capacitor_SMD:C_0603_1608Metric_Pad1.08x0.95mm_HandSolder"
+			(at 62.5348 31.75 0)
+			(effects
+				(font
+					(size 1.27 1.27)
+				)
+				(hide yes)
+			)
+		)
+		(property "Datasheet" "~"
+			(at 63.5 35.56 0)
+			(effects
+				(font
+					(size 1.27 1.27)
+				)
+				(hide yes)
+			)
+		)
+		(property "Description" "Unpolarized capacitor"
+			(at 63.5 35.56 0)
+			(effects
+				(font
+					(size 1.27 1.27)
+				)
+				(hide yes)
+			)
+		)
+		(pin "2"
+		)
+		(pin "1"
+		)
+		(instances
+			(project "BREAD_Slice"
+				(path "/66043bca-a260-4915-9fce-8a51d324c687/750db89f-8b40-4cde-930a-58e7ceb323d5"
+					(reference "C5")
+					(unit 1)
+				)
+			)
+		)
+	)
+	(symbol
 		(lib_id "Device:R")
 		(at 123.19 153.67 90)
@@
 		(on_board yes)
 		(dnp no)
-		(property "Reference" "R7"
+		(property "Reference" "R6"
 			(at 122.428 158.75 90)
 			(effects
@@
 			(project "BREAD_Slice"
 				(path "/66043bca-a260-4915-9fce-8a51d324c687/750db89f-8b40-4cde-930a-58e7ceb323d5"
-					(reference "R7")
+					(reference "R6")
 					(unit 1)
 				)
@@
 		(on_board yes)
 		(dnp no)
-		(property "Reference" "R4"
+		(property "Reference" "R7"
 			(at 122.428 165.1 90)
 			(effects
@@
 			(project "BREAD_Slice"
 				(path "/66043bca-a260-4915-9fce-8a51d324c687/750db89f-8b40-4cde-930a-58e7ceb323d5"
-					(reference "R4")
+					(reference "R7")
 					(unit 1)
 				)
