File: hardware/tps7a4901.kicad_sch (KiCad schematic)
At the start: 8 parts, among them U3 TPS7A4901DGNR

Commit message: minor tweaks
Parts:
- removed C14, C17: 10u, Capacitor_SMD:C_0805_2012Metric_Pad1.18x1.45mm_HandSolder, symbol Device:C_Small
- removed C15, C16: 10n, Capacitor_SMD:C_0805_2012Metric_Pad1.18x1.45mm_HandSolder, symbol Device:C_Small
- removed R10, R9: 99, Resistor_SMD:R_0805_2012Metric_Pad1.20x1.40mm_HandSolder, symbol Device:R
- removed U3: TPS7A4901DGNR, kml-custom:DGN8_1P89X1P57, symbol kml-custom:TPS7A4901DGNR
- added C34, C37: 10u X7R, Capacitor_SMD:C_1206_3216Metric, symbol Device:C_Small
- added C35, C36: 10n X7R, Capacitor_SMD:C_1206_3216Metric, symbol Device:C_Small
- added R27: 300k, symbol Device:R
- added R28: 100k, symbol Device:R
- added R29: 71.5k 1%, symbol Device:R
- added U8: TPS7A4901DGNR, kml-custom:DGN8_1P89X1P57, symbol kml-custom:TPS7A4901DGNR
Connections:
- net GND: now also C34.1, C35.1
- net GNDA: now also C37.1, R28.1, U8.3 (NC), U8.4 (GND), U8.EPAD
- net VAA: now also C36.2, C37.2, R27.2, U8.1 (OUT)
- net VIN: now also U8.8 (IN)
- new net: C34.2, U8.5 (EN)
- new net: C36.1, R28.2, R29.1, U8.2 (FB)
- new net: C35.2, U8.6 (NR/SS)
- new net: R27.1, R29.2
Other:
- note added: "* see notebook in documentation directory for complete calculations"
- note added: "LDO Regulator"
- note added: "VOUT = Vfb * (1 + R1/R2) R1_5V_A_CHOSEN_EQUIV = 322.000 kΩ VOUT_5V = 5.001 V"

Commit message: chore: minor updates
Parts:
- renumbered C34 to C11, C35 to C12, C36 to C13, C37 to C14, R29 to R10, R28 to R11, R27 to R9, U8 to U3
Changed lines of the file:
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@@
 		(on_board yes)
 		(dnp no)
-		(property "Reference" "C34"
+		(property "Reference" "C11"
 			(at 116.84 112.522 0)
 			(effects
@@
 			(project "BREAD_Slice"
 				(path "/66043bca-a260-4915-9fce-8a51d324c687/6de3a3fd-790e-4d94-a2c4-e38a1720a215"
-					(reference "C34")
+					(reference "C11")
 					(unit 1)
 				)
@@
 		(on_board yes)
 		(dnp no)
-		(property "Reference" "C37"
+		(property "Reference" "C14"
 			(at 205.74 96.52 0)
 			(effects
@@
 			(project "BREAD_Slice"
 				(path "/66043bca-a260-4915-9fce-8a51d324c687/6de3a3fd-790e-4d94-a2c4-e38a1720a215"
-					(reference "C37")
+					(reference "C14")
 					(unit 1)
 				)
@@
 		(on_board yes)
 		(dnp no)
-		(property "Reference" "R28"
+		(property "Reference" "R11"
 			(at 192.786 106.68 0)
 			(effects
@@
 			(project "BREAD_Slice"
 				(path "/66043bca-a260-4915-9fce-8a51d324c687/6de3a3fd-790e-4d94-a2c4-e38a1720a215"
-					(reference "R28")
+					(reference "R11")
 					(unit 1)
 				)
@@
 		(on_board yes)
 		(dnp no)
-		(property "Reference" "C35"
+		(property "Reference" "C12"
 			(at 122.682 101.854 90)
 			(effects
@@
 			(project "BREAD_Slice"
 				(path "/66043bca-a260-4915-9fce-8a51d324c687/6de3a3fd-790e-4d94-a2c4-e38a1720a215"
-					(reference "C35")
+					(reference "C12")
 					(unit 1)
 				)
@@
 		(on_board yes)
 		(dnp no)
-		(property "Reference" "R27"
+		(property "Reference" "R9"
 			(at 192.786 83.82 0)
 			(effects
@@
 			(project "BREAD_Slice"
 				(path "/66043bca-a260-4915-9fce-8a51d324c687/6de3a3fd-790e-4d94-a2c4-e38a1720a215"
-					(reference "R27")
+					(reference "R9")
 					(unit 1)
 				)
@@
 		(on_board yes)
 		(dnp no)
-		(property "Reference" "U8"
+		(property "Reference" "U3"
 			(at 151.13 87.63 0)
 			(effects
@@
 			(project "BREAD_Slice"
 				(path "/66043bca-a260-4915-9fce-8a51d324c687/6de3a3fd-790e-4d94-a2c4-e38a1720a215"
-					(reference "U8")
+					(reference "U3")
 					(unit 1)
 				)
@@
 		(dnp no)
 		(fields_autoplaced yes)
-		(property "Reference" "C36"
+		(property "Reference" "C13"
 			(at 179.07 93.9735 0)
 			(effects
@@
 			(project "BREAD_Slice"
 				(path "/66043bca-a260-4915-9fce-8a51d324c687/6de3a3fd-790e-4d94-a2c4-e38a1720a215"
-					(reference "C36")
+					(reference "C13")
 					(unit 1)
 				)
@@
 		(on_board yes)
 		(dnp no)
-		(property "Reference" "R29"
+		(property "Reference" "R10"
 			(at 192.786 93.98 0)
 			(effects
@@
 			(project "BREAD_Slice"
 				(path "/66043bca-a260-4915-9fce-8a51d324c687/6de3a3fd-790e-4d94-a2c4-e38a1720a215"
-					(reference "R29")
-					(unit 1)
-				)
+					(reference "R10")
+					(unit 1)
+				)
